Commit message: quadraped

File: body.urdf (robot description, URDF)
Before this commit: robot robot, 3 links, 2 joints
Links:
- added link BackLowerLeg, mass 1; collision box size=0.2 0.2 1; visual box size=0.2 0.2 1
- added link FrontLowerLeg, mass 1; collision box size=0.2 0.2 1; visual box size=0.2 0.2 1
- added link LeftLeg, mass 1; collision box size=1.0 0.2 0.2; visual box size=1.0 0.2 0.2
- added link LeftLowerLeg, mass 1; collision box size=0.2 0.2 1; visual box size=0.2 0.2 1
- added link RightLeg, mass 1; collision box size=1.0 0.2 0.2; visual box size=1.0 0.2 0.2
- added link RightLowerLeg, mass 1; collision box size=0.2 0.2 1; visual box size=0.2 0.2 1
- link BackLeg: geometry collision box size=0.2 1 0.2; visual box size=0.2 1 0.2
- link FrontLeg: geometry collision box size=0.2 1 0.2; visual box size=0.2 1 0.2
Joints:
- added joint BackLeg_BackLowerLeg: type revolute, parent BackLeg, child BackLowerLeg, origin xyz=0 -1 0 rpy=0 0 0, axis 1 0 0, limit lower=-3.14159 upper=3.14159 effort=0.0 velocity=0.0
- added joint FrontLeg_FrontLowerLeg: type revolute, parent FrontLeg, child FrontLowerLeg, origin xyz=0 1 0 rpy=0 0 0, axis 1 0 0, limit lower=-3.14159 upper=3.14159 effort=0.0 velocity=0.0
- added joint LeftLeg_LeftLowerLeg: type revolute, parent LeftLeg, child LeftLowerLeg, origin xyz=-1 0 0 rpy=0 0 0, axis 0 1 0, limit lower=-3.14159 upper=3.14159 effort=0.0 velocity=0.0
- added joint RightLeg_RightLowerLeg: type revolute, parent RightLeg, child RightLowerLeg, origin xyz=1 0 0 rpy=0 0 0, axis 0 1 0, limit lower=-3.14159 upper=3.14159 effort=0.0 velocity=0.0
- added joint Torso_LeftLeg: type revolute, parent Torso, child LeftLeg, origin xyz=-0.5 0 1 rpy=0 0 0, axis 0 1 0, limit lower=-3.14159 upper=3.14159 effort=0.0 velocity=0.0
- added joint Torso_RightLeg: type revolute, parent Torso, child RightLeg, origin xyz=0.5 0 1 rpy=0 0 0, axis 0 1 0, limit lower=-3.14159 upper=3.14159 effort=0.0 velocity=0.0
- joint Torso_BackLeg: axis 0 1 0 -> 1 0 0; origin xyz=0.5 0 1 rpy=0 0 0 -> xyz=0 -0.5 1 rpy=0 0 0
- joint Torso_FrontLeg: axis 0 1 0 -> 1 0 0; origin xyz=-0.5 0 1 rpy=0 0 0 -> xyz=0 0.5 1 rpy=0 0 0

Commit message: current model

File: body.urdf (robot description, URDF)
Before this commit: robot robot, 9 links, 8 joints
Links:
- link BackLeg: geometry collision box size=0.5 0.5 0.3; visual box size=0.5 0.5 0.3
- link BackLowerLeg: geometry collision box size=0.3 0.5 1; visual box size=0.3 0.5 1
- link FrontLeg: geometry collision box size=0.5 0.5 0.3; visual box size=0.5 0.5 0.3
- link FrontLowerLeg: geometry collision box size=0.3 0.5 1; visual box size=0.3 0.5 1
- link LeftLeg: geometry collision box size=0.5 0.5 0.3; visual box size=0.5 0.5 0.3
- link LeftLowerLeg: geometry collision box size=0.3 0.5 1; visual box size=0.3 0.5 1
- link RightLeg: geometry collision box size=0.5 0.5 0.3; visual box size=0.5 0.5 0.3
- link RightLowerLeg: geometry collision box size=0.3 0.5 1; visual box size=0.3 0.5 1
- link Torso: geometry collision box size=1 3 1; visual box size=1 3 1
Joints:
- joint BackLeg_BackLowerLeg: axis 1 0 0 -> 0 1 0; origin xyz=0 -1 0 rpy=0 0 0 -> xyz=0.5 -0.7 0 rpy=0 0 0
- joint FrontLeg_FrontLowerLeg: axis 1 0 0 -> 0 1 0; origin xyz=0 1 0 rpy=0 0 0 -> xyz=0.5 0.7 0 rpy=0 0 0
- joint LeftLeg_LeftLowerLeg: origin xyz=-1 0 0 rpy=0 0 0 -> xyz=-0.5 0.7 0 rpy=0 0 0
- joint RightLeg_RightLowerLeg: origin xyz=1 0 0 rpy=0 0 0 -> xyz=-0.5 -0.7 0 rpy=0 0 0
- joint Torso_BackLeg: axis 1 0 0 -> 0 1 0; origin xyz=0 -0.5 1 rpy=0 0 0 -> xyz=0.5 -0.7 1 rpy=0 0 0
- joint Torso_FrontLeg: axis 1 0 0 -> 0 1 0; origin xyz=0 0.5 1 rpy=0 0 0 -> xyz=0.5 0.7 1 rpy=0 0 0
- joint Torso_LeftLeg: origin xyz=-0.5 0 1 rpy=0 0 0 -> xyz=-0.5 0.7 1 rpy=0 0 0
- joint Torso_RightLeg: origin xyz=0.5 0 1 rpy=0 0 0 -> xyz=-0.5 -0.7 1 rpy=0 0 0

Commit message: Assignment 5

File: body.urdf (robot description, URDF)
Before this commit: robot robot, 9 links, 8 joints
Links:
- removed link FrontLeg
- removed link FrontLowerLeg
- removed link RightLeg
- removed link RightLowerLeg
- link BackLeg: geometry collision box size=0.5 3 0.3; visual box size=0.5 3 0.3
- link BackLowerLeg: geometry collision box size=0.6 3 1; visual box size=0.6 3 1
- link LeftLeg: geometry collision box size=0.5 3 0.3; visual box size=0.5 3 0.3
- link LeftLowerLeg: geometry collision box size=0.6 3 1; visual box size=0.6 3 1
- link Torso: geometry collision box size=1.5 3 1; visual box size=1.5 3 1
Joints:
- removed joint FrontLeg_FrontLowerLeg
- removed joint RightLeg_RightLowerLeg
- removed joint Torso_FrontLeg
- removed joint Torso_RightLeg
- joint BackLeg_BackLowerLeg: origin xyz=0.5 -0.7 0 rpy=0 0 0 -> xyz=0.35 -0.7 0 rpy=0 0 0
- joint LeftLeg_LeftLowerLeg: origin xyz=-0.5 0.7 0 rpy=0 0 0 -> xyz=-0.35 0.7 0 rpy=0 0 0
- joint Torso_BackLeg: origin xyz=0.5 -0.7 1 rpy=0 0 0 -> xyz=1 0 1 rpy=0 0 0
- joint Torso_LeftLeg: origin xyz=-0.5 0.7 1 rpy=0 0 0 -> xyz=-1 0 1 rpy=0 0 0

Commit message: assignment 6 snake

File: body.urdf (robot description, URDF)
Before this commit: robot robot, 5 links, 4 joints
Links:
- removed link BackLeg
- removed link BackLowerLeg
- removed link LeftLeg
- removed link LeftLowerLeg
- removed link Torso
- added link Link0, mass 1; collision box size=1.734583609760468 1.3680511530381898 0.7144741484214495; visual box size=1.734583609760468 1.3680511530381898 0.7144741484214495
- added link Link1, mass 1; collision box size=1.3195812111533873 1.543207772118189 1.8142401560229837; visual box size=1.3195812111533873 1.543207772118189 1.8142401560229837
- added link Link10, mass 1; collision box size=1.7129682613463126 1.7287016664103059 1.0794282165484297; visual box size=1.7129682613463126 1.7287016664103059 1.0794282165484297
- added link Link11, mass 1; collision box size=2.3016291142109324 0.6588181741090415 2.2743211517568085; visual box size=2.3016291142109324 0.6588181741090415 2.2743211517568085
- added link Link12, mass 1; collision box size=1.9372445637830844 1.0008225174820107 0.8068074164676209; visual box size=1.9372445637830844 1.0008225174820107 0.8068074164676209
- added link Link2, mass 1; collision box size=1.8619784031933317 2.113148618263037 0.612211566277165; visual box size=1.8619784031933317 2.113148618263037 0.612211566277165
- added link Link3, mass 1; collision box size=1.279471010554671 2.004898801224527 1.4140724616515081; visual box size=1.279471010554671 2.004898801224527 1.4140724616515081
- added link Link4, mass 1; collision box size=0.6204583938407471 1.0672603655240263 1.364469661313594; visual box size=0.6204583938407471 1.0672603655240263 1.364469661313594
- added link Link5, mass 1; collision box size=1.0735982991595643 0.9588309081599342 0.5383954285145696; visual box size=1.0735982991595643 0.9588309081599342 0.5383954285145696
- added link Link6, mass 1; collision box size=1.6111958239194661 1.1558667920705217 1.469826409055296; visual box size=1.6111958239194661 1.1558667920705217 1.469826409055296
- added link Link7, mass 1; collision box size=1.3556879340509336 0.987573475876828 1.7199632506435227; visual box size=1.3556879340509336 0.987573475876828 1.7199632506435227
- added link Link8, mass 1; collision box size=1.439331011930267 0.9805838067247512 2.051334206701992; visual box size=1.439331011930267 0.9805838067247512 2.051334206701992
- added link Link9, mass 1; collision box size=2.1834279749823784 0.5124748007894189 1.2899099092399; visual box size=2.1834279749823784 0.5124748007894189 1.2899099092399
Joints:
- removed joint BackLeg_BackLowerLeg
- removed joint LeftLeg_LeftLowerLeg
- removed joint Torso_BackLeg
- removed joint Torso_LeftLeg
- added joint Link0_Link1: type revolute, parent Link0, child Link1, origin xyz=0.867291804880234 0 2 rpy=0 0 0, axis 0 1 0, limit lower=-3.14159 upper=3.14159 effort=0.0 velocity=0.0
- added joint Link10_Link11: type revolute, parent Link10, child Link11, origin xyz=1.7129682613463126 0 0 rpy=0 0 0, axis 0 1 0, limit lower=-3.14159 upper=3.14159 effort=0.0 velocity=0.0
- added joint Link11_Link12: type revolute, parent Link11, child Link12, origin xyz=2.3016291142109324 0 0 rpy=0 0 0, axis 0 1 0, limit lower=-3.14159 upper=3.14159 effort=0.0 velocity=0.0
- added joint Link1_Link2: type revolute, parent Link1, child Link2, origin xyz=1.3195812111533873 0 0 rpy=0 0 0, axis 0 1 0, limit lower=-3.14159 upper=3.14159 effort=0.0 velocity=0.0
- added joint Link2_Link3: type revolute, parent Link2, child Link3, origin xyz=1.8619784031933317 0 0 rpy=0 0 0, axis 0 1 0, limit lower=-3.14159 upper=3.14159 effort=0.0 velocity=0.0
- added joint Link3_Link4: type revolute, parent Link3, child Link4, origin xyz=1.279471010554671 0 0 rpy=0 0 0, axis 0 1 0, limit lower=-3.14159 upper=3.14159 effort=0.0 velocity=0.0
- added joint Link4_Link5: type revolute, parent Link4, child Link5, origin xyz=0.6204583938407471 0 0 rpy=0 0 0, axis 0 1 0, limit lower=-3.14159 upper=3.14159 effort=0.0 velocity=0.0
- added joint Link5_Link6: type revolute, parent Link5, child Link6, origin xyz=1.0735982991595643 0 0 rpy=0 0 0, axis 0 1 0, limit lower=-3.14159 upper=3.14159 effort=0.0 velocity=0.0
- added joint Link6_Link7: type revolute, parent Link6, child Link7, origin xyz=1.6111958239194661 0 0 rpy=0 0 0, axis 0 1 0, limit lower=-3.14159 upper=3.14159 effort=0.0 velocity=0.0
- added joint Link7_Link8: type revolute, parent Link7, child Link8, origin xyz=1.3556879340509336 0 0 rpy=0 0 0, axis 0 1 0, limit lower=-3.14159 upper=3.14159 effort=0.0 velocity=0.0
- added joint Link8_Link9: type revolute, parent Link8, child Link9, origin xyz=1.439331011930267 0 0 rpy=0 0 0, axis 0 1 0, limit lower=-3.14159 upper=3.14159 effort=0.0 velocity=0.0
- added joint Link9_Link10: type revolute, parent Link9, child Link10, origin xyz=2.1834279749823784 0 0 rpy=0 0 0, axis 0 1 0, limit lower=-3.14159 upper=3.14159 effort=0.0 velocity=0.0

Commit message: wip assignment7

File: body.urdf (robot description, URDF)
Before this commit: robot robot, 13 links, 12 joints
Links:
- removed link Link10
- removed link Link11
- removed link Link12
- removed link Link9
- link Link0: geometry collision box size=1.7439291333450475 1.386862398925972 1.4383568809291352; visual box size=1.7439291333450475 1.386862398925972 1.4383568809291352
- link Link1: geometry collision box size=1.092528408481146 1.9104443155109452 0.6398737353733417; visual box size=1.092528408481146 1.9104443155109452 0.6398737353733417
- link Link2: geometry collision box size=1.495038242827999 1.8441665045505118 1.4794282943870787; visual box size=1.495038242827999 1.8441665045505118 1.4794282943870787
- link Link3: geometry collision box size=0.9948614779120649 1.286192577691901 0.530304101077683; visual box size=0.9948614779120649 1.286192577691901 0.530304101077683
- link Link4: geometry collision box size=1.001513665002201 0.5916059768868334 1.0122282627740309; visual box size=1.001513665002201 0.5916059768868334 1.0122282627740309
- link Link5: geometry collision box size=0.9685154979894045 0.6927165651386484 1.840994593250497; visual box size=0.9685154979894045 0.6927165651386484 1.840994593250497
- link Link6: geometry collision box size=0.9392013400055419 0.8694622904902641 1.149733207878058; visual box size=0.9392013400055419 0.8694622904902641 1.149733207878058
- link Link7: geometry collision box size=1.9330681524795643 0.7342668355355146 1.7095003224352932; visual box size=1.9330681524795643 0.7342668355355146 1.7095003224352932
- link Link8: geometry collision box size=1.0495022396631946 1.9006571041349332 1.6816694346242778; visual box size=1.0495022396631946 1.9006571041349332 1.6816694346242778
Joints:
- removed joint Link10_Link11
- removed joint Link11_Link12
- removed joint Link2_Link3
- removed joint Link5_Link6
- removed joint Link6_Link7
- removed joint Link7_Link8
- removed joint Link8_Link9
- removed joint Link9_Link10
- added joint Link0_Link3: type revolute, parent Link0, child Link3, origin xyz=0 0.693431199462986 2 rpy=0 0 0, axis 1 0 0, limit lower=-3.14159 upper=3.14159 effort=0.0 velocity=0.0
- added joint Link1_Link6: type revolute, parent Link1, child Link6, origin xyz=-1.092528408481146 0 0 rpy=0 0 0, axis 0 1 0, limit lower=-3.14159 upper=3.14159 effort=0.0 velocity=0.0
- added joint Link1_Link8: type revolute, parent Link1, child Link8, origin xyz=0 0 -0.6398737353733417 rpy=0 0 0, axis 0 0 1, limit lower=-3.14159 upper=3.14159 effort=0.0 velocity=0.0
- added joint Link4_Link7: type revolute, parent Link4, child Link7, origin xyz=-1.001513665002201 0 0 rpy=0 0 0, axis 0 1 0, limit lower=-3.14159 upper=3.14159 effort=0.0 velocity=0.0
- joint Link0_Link1: axis 0 1 0 -> 1 0 0; origin xyz=0.867291804880234 0 2 rpy=0 0 0 -> xyz=0 -0.693431199462986 2 rpy=0 0 0
- joint Link1_Link2: origin xyz=1.3195812111533873 0 0 rpy=0 0 0 -> xyz=1.092528408481146 0 0 rpy=0 0 0
- joint Link3_Link4: axis 0 1 0 -> 0 0 1; origin xyz=1.279471010554671 0 0 rpy=0 0 0 -> xyz=0 0 -0.530304101077683 rpy=0 0 0
- joint Link4_Link5: axis 0 1 0 -> 0 0 1; origin xyz=0.6204583938407471 0 0 rpy=0 0 0 -> xyz=0 0 -1.0122282627740309 rpy=0 0 0

Commit message: wip assignment 7 pt 2

File: body.urdf (robot description, URDF)
Before this commit: robot robot, 9 links, 8 joints
Links:
- removed link Link8
- link Link0: geometry collision box size=0.5056620950070545 1.258921522916528 0.6353658631672805; visual box size=0.5056620950070545 1.258921522916528 0.6353658631672805
- link Link1: geometry collision box size=0.7139151399198491 1.2074860740744877 0.8034478491790319; visual box size=0.7139151399198491 1.2074860740744877 0.8034478491790319
- link Link2: geometry collision box size=0.6844359186023091 0.708677825483234 1.2719228275707886; visual box size=0.6844359186023091 0.708677825483234 1.2719228275707886
- link Link3: geometry collision box size=0.7065857161823288 1.4574236718355107 0.7341804943313459; visual box size=0.7065857161823288 1.4574236718355107 0.7341804943313459
- link Link4: geometry collision box size=1.0643175558565758 1.3016349778569618 1.8009339135260922; visual box size=1.0643175558565758 1.3016349778569618 1.8009339135260922
- link Link5: geometry collision box size=1.8308074886916925 1.057355590586754 1.4035663317724874; visual box size=1.8308074886916925 1.057355590586754 1.4035663317724874
- link Link6: geometry collision box size=1.563425594612151 0.8551316972836217 0.8467740172566289; visual box size=1.563425594612151 0.8551316972836217 0.8467740172566289
- link Link7: geometry collision box size=1.3303246530095663 1.1165375287204582 1.7455980329495095; visual box size=1.3303246530095663 1.1165375287204582 1.7455980329495095
Joints:
- removed joint Link0_Link3
- removed joint Link1_Link2
- removed joint Link1_Link6
- removed joint Link1_Link8
- removed joint Link4_Link5
- removed joint Link4_Link7
- added joint Link0_Link2: type revolute, parent Link0, child Link2, origin xyz=-0.25283104750352725 0 2 rpy=0 0 0, axis 0 1 0, limit lower=-3.14159 upper=3.14159 effort=0.0 velocity=0.0
- added joint Link0_Link5: type revolute, parent Link0, child Link5, origin xyz=0.25283104750352725 0 2 rpy=0 0 0, axis 0 1 0, limit lower=-3.14159 upper=3.14159 effort=0.0 velocity=0.0
- added joint Link0_Link6: type revolute, parent Link0, child Link6, origin xyz=0 -0.629460761458264 2 rpy=0 0 0, axis 1 0 0, limit lower=-3.14159 upper=3.14159 effort=0.0 velocity=0.0
- added joint Link1_Link7: type revolute, parent Link1, child Link7, origin xyz=0 0 0.8034478491790319 rpy=0 0 0, axis 0 0 1, limit lower=-3.14159 upper=3.14159 effort=0.0 velocity=0.0
- added joint Link2_Link3: type revolute, parent Link2, child Link3, origin xyz=-0.6844359186023091 0 0 rpy=0 0 0, axis 0 1 0, limit lower=-3.14159 upper=3.14159 effort=0.0 velocity=0.0
- joint Link0_Link1: origin xyz=0 -0.693431199462986 2 rpy=0 0 0 -> xyz=0 0.629460761458264 2 rpy=0 0 0
- joint Link3_Link4: axis 0 0 1 -> 0 1 0; origin xyz=0 0 -0.530304101077683 rpy=0 0 0 -> xyz=0 1.4574236718355107 0 rpy=0 0 0

Commit message: Assignment 7

File: body.urdf (robot description, URDF)
Before this commit: robot robot, 8 links, 7 joints
Links:
- added link Link8, mass 1; collision box size=0.5065675725500132 0.8797011484567681 1.1978461520120551; visual box size=0.5065675725500132 0.8797011484567681 1.1978461520120551
- link Link0: geometry collision box size=1.7248002286248338 0.6489323977667989 1.7094995568532982; visual box size=1.7248002286248338 0.6489323977667989 1.7094995568532982
- link Link1: geometry collision box size=1.0882581562329345 1.6719702008311972 0.6978348393617294; visual box size=1.0882581562329345 1.6719702008311972 0.6978348393617294
- link Link2: geometry collision box size=1.286053169935478 1.6579857644141862 0.9799520929256652; visual box size=1.286053169935478 1.6579857644141862 0.9799520929256652
- link Link3: geometry collision box size=1.8178203191648556 1.6636463741422276 0.650831411369375; visual box size=1.8178203191648556 1.6636463741422276 0.650831411369375
- link Link4: geometry collision box size=0.5139752088841953 1.6571296614555204 1.0840576085904845; visual box size=0.5139752088841953 1.6571296614555204 1.0840576085904845
- link Link5: geometry collision box size=1.8725986968084811 1.2316286523670708 0.8480054178214795; visual box size=1.8725986968084811 1.2316286523670708 0.8480054178214795
- link Link6: geometry collision box size=1.1975096265214933 1.5613931310850229 1.55739036415932; visual box size=1.1975096265214933 1.5613931310850229 1.55739036415932
- link Link7: geometry collision box size=1.8357056356724066 1.3152464936693713 0.9824248653515404; visual box size=1.8357056356724066 1.3152464936693713 0.9824248653515404
Joints:
- removed joint Link0_Link2
- removed joint Link0_Link5
- removed joint Link0_Link6
- removed joint Link1_Link7
- removed joint Link2_Link3
- removed joint Link3_Link4
- added joint Link0_Link3: type revolute, parent Link0, child Link3, origin xyz=0 -0.32446619888339945 2 rpy=0 0 0, axis 1 0 0, limit lower=-3.14159 upper=3.14159 effort=0.0 velocity=0.0
- added joint Link1_Link2: type revolute, parent Link1, child Link2, origin xyz=0.5441290781164673 0.8359851004155986 0 rpy=0 0 0, axis 0 1 0, limit lower=-3.14159 upper=3.14159 effort=0.0 velocity=0.0
- added joint Link1_Link4: type revolute, parent Link1, child Link4, origin xyz=1.6719702008311972 0 0 rpy=0 0 0, axis 0 1 0, limit lower=-3.14159 upper=3.14159 effort=0.0 velocity=0.0
- added joint Link1_Link5: type revolute, parent Link1, child Link5, origin xyz=-0.5441290781164673 0.8359851004155986 0 rpy=0 0 0, axis 0 1 0, limit lower=-3.14159 upper=3.14159 effort=0.0 velocity=0.0
- added joint Link3_Link6: type revolute, parent Link3, child Link6, origin xyz=0.9089101595824278 -0.8318231870711138 0 rpy=0 0 0, axis 0 1 0, limit lower=-3.14159 upper=3.14159 effort=0.0 velocity=0.0
- added joint Link5_Link7: type revolute, parent Link5, child Link7, origin xyz=-1.8725986968084811 0 0 rpy=0 0 0, axis 0 1 0, limit lower=-3.14159 upper=3.14159 effort=0.0 velocity=0.0
- added joint Link6_Link8: type revolute, parent Link6, child Link8, origin xyz=0.5987548132607466 0 0.77869518207966 rpy=0 0 0, axis 0 0 1, limit lower=-3.14159 upper=3.14159 effort=0.0 velocity=0.0
- joint Link0_Link1: origin xyz=0 0.629460761458264 2 rpy=0 0 0 -> xyz=0 0.32446619888339945 2 rpy=0 0 0

Commit message: Assignment7

File: body.urdf (robot description, URDF)
Before this commit: robot robot, 9 links, 8 joints
Links:
- link Link0: geometry collision box size=1.0820530997638091 1.0554737301106198 0.9024091736405127; visual box size=1.0820530997638091 1.0554737301106198 0.9024091736405127
- link Link1: geometry collision box size=0.9450934068210565 1.0696743737410495 0.8180628127819374; visual box size=0.9450934068210565 1.0696743737410495 0.8180628127819374
- link Link2: geometry collision box size=0.8918839378260162 1.6100436670161573 1.8797300027797856; visual box size=0.8918839378260162 1.6100436670161573 1.8797300027797856
- link Link3: geometry collision box size=0.6452709558052551 1.8587366633976679 0.6100205162442184; visual box size=0.6452709558052551 1.8587366633976679 0.6100205162442184
- link Link4: geometry collision box size=1.0184029784990474 1.8676921129066888 1.6631225664493485; visual box size=1.0184029784990474 1.8676921129066888 1.6631225664493485
- link Link5: geometry collision box size=1.1116897811988058 0.7599241385662169 1.3124986010722357; visual box size=1.1116897811988058 0.7599241385662169 1.3124986010722357
- link Link6: geometry collision box size=1.569739850045098 1.4492548918338861 0.868240852388972; visual box size=1.569739850045098 1.4492548918338861 0.868240852388972
- link Link7: geometry collision box size=1.034488696660814 1.187544597080068 0.9787417295322958; visual box size=1.034488696660814 1.187544597080068 0.9787417295322958
- link Link8: geometry collision box size=0.9814653312903152 1.500905163874199 0.892711063678802; visual box size=0.9814653312903152 1.500905163874199 0.892711063678802
Joints:
- removed joint Link0_Link3
- removed joint Link1_Link4
- removed joint Link1_Link5
- removed joint Link3_Link6
- removed joint Link5_Link7
- removed joint Link6_Link8
- added joint Link1_Link3: type revolute, parent Link1, child Link3, origin xyz=0.47254670341052823 -0.5348371868705247 0 rpy=0 0 0, axis 0 1 0, limit lower=-3.14159 upper=3.14159 effort=0.0 velocity=0.0
- added joint Link2_Link4: type revolute, parent Link2, child Link4, origin xyz=0.4459419689130081 -0.8050218335080787 0 rpy=0 0 0, axis 0 1 0, limit lower=-3.14159 upper=3.14159 effort=0.0 velocity=0.0
- added joint Link2_Link5: type revolute, parent Link2, child Link5, origin xyz=0.8918839378260162 0 0 rpy=0 0 0, axis 0 1 0, limit lower=-3.14159 upper=3.14159 effort=0.0 velocity=0.0
- added joint Link2_Link6: type revolute, parent Link2, child Link6, origin xyz=0.4459419689130081 0.8050218335080787 0 rpy=0 0 0, axis 0 1 0, limit lower=-3.14159 upper=3.14159 effort=0.0 velocity=0.0
- added joint Link4_Link7: type revolute, parent Link4, child Link7, origin xyz=0 -0.9338460564533444 0.8315612832246743 rpy=0 0 0, axis 0 0 1, limit lower=-3.14159 upper=3.14159 effort=0.0 velocity=0.0
- added joint Link7_Link8: type revolute, parent Link7, child Link8, origin xyz=0 0 0.9787417295322958 rpy=0 0 0, axis 0 0 1, limit lower=-3.14159 upper=3.14159 effort=0.0 velocity=0.0
- joint Link0_Link1: axis 1 0 0 -> 0 1 0; origin xyz=0 0.32446619888339945 2 rpy=0 0 0 -> xyz=0.5410265498819046 0 2 rpy=0 0 0
- joint Link1_Link2: origin xyz=0.5441290781164673 0.8359851004155986 0 rpy=0 0 0 -> xyz=0.9450934068210565 0 0 rpy=0 0 0
