Commit message: Assignment7

File: body.urdf (robot description, URDF)
Before this commit: robot robot, 9 links, 8 joints
Links:
- removed link Link8
- link Link0: geometry collision box size=0.5269733210035155 1.7197210694644882 0.5456640564359205; visual box size=0.5269733210035155 1.7197210694644882 0.5456640564359205
- link Link1: geometry collision box size=1.0487465997639993 1.9587207628471794 1.695929906458861; visual box size=1.0487465997639993 1.9587207628471794 1.695929906458861
- link Link2: geometry collision box size=1.0343213795464106 1.1220549407902038 1.0353040787654013; visual box size=1.0343213795464106 1.1220549407902038 1.0353040787654013
- link Link3: geometry collision box size=1.168819881705957 0.8090081555618974 1.5039916999777394; visual box size=1.168819881705957 0.8090081555618974 1.5039916999777394
- link Link4: geometry collision box size=0.8748292632520451 0.7556549902400986 1.4997836609586424; visual box size=0.8748292632520451 0.7556549902400986 1.4997836609586424
- link Link5: geometry collision box size=1.950584027815017 0.6377055945073771 1.5754554069702529; visual box size=1.950584027815017 0.6377055945073771 1.5754554069702529
- link Link6: geometry collision box size=0.5356653132357019 1.5727929332200457 0.8683626797658361; visual box size=0.5356653132357019 1.5727929332200457 0.8683626797658361
- link Link7: geometry collision box size=0.8559096653413817 1.9122536760311626 1.7710109960570857; visual box size=0.8559096653413817 1.9122536760311626 1.7710109960570857
Joints:
- removed joint Link1_Link3
- removed joint Link2_Link5
- removed joint Link2_Link6
- removed joint Link4_Link7
- removed joint Link7_Link8
- added joint Link0_Link3: type revolute, parent Link0, child Link3, origin xyz=0 0 2.27283202821796 rpy=0 0 0, axis 0 0 1, limit lower=-3.14159 upper=3.14159 effort=0.0 velocity=0.0
- added joint Link0_Link6: type revolute, parent Link0, child Link6, origin xyz=0 0.8598605347322441 2 rpy=0 0 0, axis 1 0 0, limit lower=-3.14159 upper=3.14159 effort=0.0 velocity=0.0
- added joint Link3_Link5: type revolute, parent Link3, child Link5, origin xyz=0.5844099408529785 0 0.7519958499888697 rpy=0 0 0, axis 0 1 0, limit lower=-3.14159 upper=3.14159 effort=0.0 velocity=0.0
- added joint Link6_Link7: type revolute, parent Link6, child Link7, origin xyz=-0.26783265661785094 0.7863964666100228 0 rpy=0 0 0, axis 0 1 0, limit lower=-3.14159 upper=3.14159 effort=0.0 velocity=0.0
- joint Link0_Link1: axis 0 1 0 -> 1 0 0; origin xyz=0.5410265498819046 0 2 rpy=0 0 0 -> xyz=0 -0.8598605347322441 2 rpy=0 0 0
- joint Link1_Link2: origin xyz=0.9450934068210565 0 0 rpy=0 0 0 -> xyz=0 -1.9587207628471794 0 rpy=0 0 0
- joint Link2_Link4: origin xyz=0.4459419689130081 -0.8050218335080787 0 rpy=0 0 0 -> xyz=0 -1.1220549407902038 0 rpy=0 0 0

Commit message: Assignment 7

File: body.urdf (robot description, URDF)
Before this commit: robot robot, 8 links, 7 joints
Links:
- added link Link8, mass 1; collision box size=1.193518035553594 1.3900309597455336 1.9084115079039194; visual box size=1.193518035553594 1.3900309597455336 1.9084115079039194
- added link Link9, mass 1; collision box size=1.3537198651326392 1.7460549889135444 1.8249842362550863; visual box size=1.3537198651326392 1.7460549889135444 1.8249842362550863
- link Link0: geometry collision box size=1.9939490635859975 0.8158652812176852 0.5456176613705723; visual box size=1.9939490635859975 0.8158652812176852 0.5456176613705723
- link Link1: geometry collision box size=1.465510170929416 1.4634154819260041 1.8655486085511144; visual box size=1.465510170929416 1.4634154819260041 1.8655486085511144
- link Link2: geometry collision box size=0.6649682693134438 1.179295749812048 1.5523797870931408; visual box size=0.6649682693134438 1.179295749812048 1.5523797870931408
- link Link3: geometry collision box size=1.2808939602727178 1.91413831014703 0.6305961080717137; visual box size=1.2808939602727178 1.91413831014703 0.6305961080717137
- link Link4: geometry collision box size=1.6742575870637513 0.7609195829234539 1.5874993460387978; visual box size=1.6742575870637513 0.7609195829234539 1.5874993460387978
- link Link5: geometry collision box size=1.9900082847192682 0.6204331584130669 0.5965227658545645; visual box size=1.9900082847192682 0.6204331584130669 0.5965227658545645
- link Link6: geometry collision box size=1.8593682444629869 1.056743476568964 1.0237172816471558; visual box size=1.8593682444629869 1.056743476568964 1.0237172816471558
- link Link7: geometry collision box size=1.5035632847954603 0.7009791873479048 1.5353080486570911; visual box size=1.5035632847954603 0.7009791873479048 1.5353080486570911
Joints:
- removed joint Link0_Link6
- removed joint Link2_Link4
- removed joint Link6_Link7
- added joint Link1_Link6: type revolute, parent Link1, child Link6, origin xyz=0.732755085464708 -0.7317077409630021 0 rpy=0 0 0, axis 0 1 0, limit lower=-3.14159 upper=3.14159 effort=0.0 velocity=0.0
- added joint Link1_Link9: type revolute, parent Link1, child Link9, origin xyz=0 -1.4634154819260041 0 rpy=0 0 0, axis 0 1 0, limit lower=-3.14159 upper=3.14159 effort=0.0 velocity=0.0
- added joint Link3_Link4: type revolute, parent Link3, child Link4, origin xyz=-0.6404469801363589 0.957069155073515 0 rpy=0 0 0, axis 0 1 0, limit lower=-3.14159 upper=3.14159 effort=0.0 velocity=0.0
- added joint Link4_Link7: type revolute, parent Link4, child Link7, origin xyz=-1.6742575870637513 0 0 rpy=0 0 0, axis 0 1 0, limit lower=-3.14159 upper=3.14159 effort=0.0 velocity=0.0
- added joint Link6_Link8: type revolute, parent Link6, child Link8, origin xyz=0.9296841222314934 -0.528371738284482 0 rpy=0 0 0, axis 0 1 0, limit lower=-3.14159 upper=3.14159 effort=0.0 velocity=0.0
- joint Link0_Link1: origin xyz=0 -0.8598605347322441 2 rpy=0 0 0 -> xyz=0 -0.4079326406088426 2 rpy=0 0 0
- joint Link0_Link3: axis 0 0 1 -> 1 0 0; origin xyz=0 0 2.27283202821796 rpy=0 0 0 -> xyz=0 0.4079326406088426 2 rpy=0 0 0
- joint Link1_Link2: origin xyz=0 -1.9587207628471794 0 rpy=0 0 0 -> xyz=-0.732755085464708 -0.7317077409630021 0 rpy=0 0 0
- joint Link3_Link5: origin xyz=0.5844099408529785 0 0.7519958499888697 rpy=0 0 0 -> xyz=0.6404469801363589 0.957069155073515 0 rpy=0 0 0
